File: QuadPowerDistro v0.brd (EAGLE design)
At the start: 50 x 50 mm, 17 parts, among them IC1 INA169, X1 XT60, X2 XT60, X3 XT60, X4 XT60, X5 XT60

Commit message: File updates
Making the filenames clearer.
Other:
- board text added: "Wires and Bits"
- board text added: "v0"
Changed lines of the file:
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@@
 <text x="22.86" y="13.97" size="1.778" layer="25">+ in</text>
 <text x="20.955" y="34.29" size="1.778" layer="25">- in</text>
+<text x="12.7" y="2.54" size="1.778" layer="21" rot="R90">Wires and Bits</text>
+<text x="46.99" y="20.32" size="1.778" layer="21" rot="R90">v0</text>
 </plain>
 <attributes>

Commit message: Adding more information.
Changed lines of the file:
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@@
 <text x="20.955" y="34.29" size="1.778" layer="25">- in</text>
 <text x="12.7" y="2.54" size="1.778" layer="21" rot="R90">Wires and Bits</text>
-<text x="46.99" y="20.32" size="1.778" layer="21" rot="R90">v0</text>
+<text x="22.86" y="2.54" size="1.778" layer="21" rot="R90">v0</text>
 </plain>
 <attributes>
