File: QuadPowerDistro v0.sch (EAGLE design)
At the start: 17 parts, among them IC1 INA169, X1 XT60, X2 XT60, X3 XT60, X4 XT60, X5 XT60

Commit message: File updates
Making the filenames clearer.
Other:
- note added: "http://www.wiresandbits.co.uk"
- note added: "https://github.com/pinski1/QuadcopterPowerDistro"
Changed lines of the file:
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@@
 +50V max
 +180A peak</text>
+<text x="162.56" y="35.56" size="2.54" layer="97">http://www.wiresandbits.co.uk</text>
+<text x="162.56" y="30.48" size="2.54" layer="97">https://github.com/pinski1/QuadcopterPowerDistro</text>
 </plain>
 <instances>

Commit message: Adding more information.
Other:
- note added: "https://github.com/pinski1/QuadPowerDistro"
- note removed: "https://github.com/pinski1/QuadcopterPowerDistro"
Changed lines of the file:
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@@
 +180A peak</text>
 <text x="162.56" y="35.56" size="2.54" layer="97">http://www.wiresandbits.co.uk</text>
-<text x="162.56" y="30.48" size="2.54" layer="97">https://github.com/pinski1/QuadcopterPowerDistro</text>
+<text x="162.56" y="30.48" size="2.54" layer="97">https://github.com/pinski1/QuadPowerDistro</text>
 </plain>
 <instances>
